File: kicad/infnoise_goldfingers.kicad_pcb (KiCad board)
At the start: 2 copper layers, 34.8 x 12.2 mm, 28 parts, among them SW1 MC74VHC1G66DFT1G, SW2 MC74VHC1G66DFT1G, X1 USBRAWPINS

Commit message: add 3D models
Routing:
- net GND: vias 11 -> 1
- net (no net): vias 0 -> 10

Commit message: finished assigning models to PCB
Routing:
- net /USB_P: track 8.67 -> 14.7 mm
- net /USB_M: track 8.57 -> 2.50 mm
Changed lines of the file:
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@@
   (general
     (links 66)
-    (no_connects 5)
+    (no_connects 9)
     (area 131.001699 98.832599 166.000501 111.174601)
     (thickness 1.6)
@@
   (page A4)
   (layers
-    (0 Top signal hide)
-    (31 Bottom signal hide)
+    (0 Top signal)
+    (31 Bottom signal)
     (32 B.Adhes user hide)
     (33 F.Adhes user hide)
@@
     (pad 4 smd rect (at 0.65 -0.85 90) (size 0.35 0.8) (layers Top F.Paste F.Mask)
       (net 18 /SW1EN))
+    (model TO_SOT_Packages_SMD.3dshapes/SOT-353_SC-70-5.wrl
+      (at (xyz 0 0 0))
+      (scale (xyz 1 1 1))
+      (rotate (xyz 0 0 -90))
+    )
   )
   (module SC70-5L (layer Top)
@@
     (pad 4 smd rect (at 0.65 -0.85 90) (size 0.35 0.8) (layers Top F.Paste F.Mask)
       (net 19 /SW2EN))
+    (model TO_SOT_Packages_SMD.3dshapes/SOT-353_SC-70-5.wrl
+      (at (xyz 0 0 0))
+      (scale (xyz 1 1 1))
+      (rotate (xyz 0 0 -90))
+    )
   )
   (module 0603-CAP (layer Top)
@@
   (segment (start 136.4567 104.0036) (end 136.5329 104.0036) (width 0.254) (layer Top) (net 11))
   (segment (start 136.5329 104.0036) (end 136.5329 103.9274) (width 0.254) (layer Top) (net 11))
+  (segment (start 136.5329 105.9274) (end 142.4505 105.9274) (width 0.3048) (layer Top) (net 11))
+  (segment (start 136.4567 106.0036) (end 136.5329 106.0036) (width 0.254) (layer Top) (net 11))
+  (segment (start 136.5329 106.0036) (end 136.5329 105.9274) (width 0.254) (layer Top) (net 11))
   (segment (start 142.4505 105.9274) (end 142.4505 108.4274) (width 0.254) (layer Top) (net 12))
-  (segment (start 136.5329 105.9274) (end 142.4505 105.9274) (width 0.3048) (layer Top) (net 12))
-  (segment (start 136.4567 106.0036) (end 136.5329 106.0036) (width 0.254) (layer Top) (net 12))
-  (segment (start 136.5329 106.0036) (end 136.5329 105.9274) (width 0.254) (layer Top) (net 12))
   (segment (start 152.4255 107.8274) (end 152.4255 105.7774) (width 0.254) (layer Top) (net 13))
   (via (at 151.1755 106.9274) (size 0.6858) (drill 0.3302) (layers Top Bottom) (net 13))
